File: hardware/sem-tanfolyam-stc-panel.kicad_sch (KiCad schematic)
At the start: 25 parts

Commit message: Add peripherals to schematic and 7-segment display symbol and footprint
Parts:
- added D4, D5, D6: RED, symbol Device:LED_Filled
- added R10, R11, R12, R14, R15, R16, R20, R21, R22, R8, R9: 1k, symbol Device:R
- added R17: R_Photo, symbol Device:R_Photo
- added R18, R19: 10k, symbol Device:R
- added R23: R, symbol Device:R
- added SW2, SW3: SW_Push, symbol Switch:SW_Push
- added U2: SN420362N, sem-tanfolyam:SN420362N, symbol sem-tanfolyam:SN420362N
- added U3: 74HC595, symbol 74xx:74HC595
- gave numbers to parts that had none: 25
Connections:
- net GND: now also D4.1 (K), D5.1 (K), D6.1 (K), R23.2, SW2.2, SW3.2, U3.13 (~{OE}), U3.8 (GND)
- net VCC: now also R17.1, R18.1, R19.1, U3.10 (~{SRCLR}), U3.16 (VCC)
- new net: R9.1, U3.1 (QB)
- new net: R9.2, U2.9 (B)
- new net: D4.2 (A), R20.2
- new net: R16.1, U3.7 (QH)
- new net: R16.2, U2.2 (DP)
- new net: R8.1, U3.15 (QA)
- new net: R10.1, U3.2 (QC)
- new net: R11.1, U3.3 (QD)
- new net: R12.1, U3.4 (QE)
- new net: R14.1, U3.5 (QF)
- new net: R15.1, U3.6 (QG)
- new net: R12.2, U2.7 (E)
- new net: D6.2 (A), R22.2
- new net: D5.2 (A), R21.2
- new net: R14.2, U2.4 (F)
- new net: R10.2, U2.8 (C)
- new net: R8.2, U2.3 (A)
- new net: R15.2, U2.1 (G)
- new net: R11.2, U2.6 (D)
- new net ADC: R17.2, R23.1
- new net BTN0: R18.2, SW2.1
- new net BTN1: R19.2, SW3.1
- new net CLK: U3.11 (SRCLK)
- new net DIG1: U2.10 (DIG.1)
- new net DIG2: U2.5 (DIG.2)
- new net LATCH: U3.12 (RCLK)
- new net LED0: R20.1
- new net LED1: R21.1
- new net LED2: R22.1
- new net SD: U3.14 (SER)
- no-connect marks 7 -> 8
Other:
- note added: "Pins to assign:"
- moved on the sheet: U4

Commit message: Add PCB design
Parts:
- removed C3, C4: 27pF, symbol Device:C
- removed D6: RED, symbol Device:LED_Filled
- removed J1: USB_B_Micro, symbol Connector:USB_B_Micro
- removed R10, R14, R15, R16, R20, R21, R22: 1k, symbol Device:R
- removed R17: R_Photo, symbol Device:R_Photo
- removed R18, R19: 10k, symbol Device:R
- removed R23: R, symbol Device:R
- removed SW2, SW3: SW_Push, symbol Switch:SW_Push
- removed U1: CH340G, Package_SO:SOIC-16_3.9x9.9mm_P1.27mm, symbol Interface_USB:CH340G
- removed U2: SN420362N, sem-tanfolyam:SN420362N, symbol sem-tanfolyam:SN420362N
- removed U3: 74HC595, symbol 74xx:74HC595
- removed Y1: 12 MHz, symbol Device:Crystal
- added J1, J2: Conn_01x09_Male, Connector_PinHeader_2.54mm:PinHeader_1x09_P2.54mm_Vertical, symbol Connector:Conn_01x09_Male
- added J3: USB_C_Receptacle_USB2.0, Connector_USB:USB_C_Receptacle_G-Switch_GT-USB-7010ASV, symbol Connector:USB_C_Receptacle_USB2.0
- added U1: CH340E, Package_SO:MSOP-10_3x3mm_P0.5mm, symbol Interface_USB:CH340E
- C1: renamed from C6; footprint (none) -> Capacitor_SMD:C_0603_1608Metric
- C2: renamed from C1; footprint (none) -> Capacitor_SMD:C_0603_1608Metric
- C3: renamed from C5; footprint (none) -> Capacitor_SMD:C_0603_1608Metric
- C4: renamed from C2; footprint (none) -> Capacitor_SMD:C_0603_1608Metric
- D1: renamed from D2; footprint (none) -> Diode_SMD:D_MiniMELF
- D2: renamed from D1; footprint (none) -> Diode_SMD:D_MiniMELF
- D3: footprint (none) -> LED_SMD:LED_0603_1608Metric
- D4: value RED -> ACT; footprint (none) -> LED_SMD:LED_0603_1608Metric
- D5: value RED -> USER; footprint (none) -> LED_SMD:LED_0603_1608Metric
- F1: footprint (none) -> Fuse:Fuse_1206_3216Metric
- R1: renamed from R5; footprint (none) -> Resistor_SMD:R_0603_1608Metric
- R10: renamed from R4; footprint (none) -> Resistor_SMD:R_0603_1608Metric
- R11, R12, R6, R7: footprint (none) -> Resistor_SMD:R_0603_1608Metric
- R2: renamed from R1; footprint (none) -> Resistor_SMD:R_0603_1608Metric
- R3: renamed from R2; footprint (none) -> Resistor_SMD:R_0603_1608Metric
- R4: renamed from R13; footprint (none) -> Resistor_SMD:R_0603_1608Metric
- R5: renamed from R3; footprint (none) -> Resistor_SMD:R_0603_1608Metric
- R8, R9: value 1k -> 5k1; footprint (none) -> Resistor_SMD:R_0603_1608Metric
- SW1: footprint (none) -> Button_Switch_SMD:SW_Push_1P1T_NO_6x6mm_H9.5mm
- U2: renamed from U4; footprint (none) -> Package_SO:TSSOP-20_4.4x6.5mm_P0.65mm
- renumbered Q2 to Q1, Q1 to Q2
Connections:
- net GND: now also R8.2, R9.2, J2.9 (Pin_9), J3.A1 (GND), J3.A12 (GND), J3.B1 (GND), J3.B12 (GND), J3.S1 (SHIELD), U1.3 (GND)
- net RST: now also J1.9 (Pin_9)
- net USB_DM: now also J3.A7 (D-), J3.B7 (D-), U1.2 (UD-)
- net USB_DP: now also J3.A6 (D+), J3.B6 (D+), U1.1 (UD+)
- net VBUS: now also U1.7 (VCC)
- net VCC: now also J2.8 (Pin_8)
- net at R9.1: now also J3.A5 (CC1)
- net at D4.2 (A): now also R11.2
- net at R1.2: now also U1.9 (RXD)
- net at R8.1: now also J3.B5 (CC2)
- net at R11.1: now also U1.6 (TNOW)
- net P5.5: now reaches R12.1
- net P5.5: now also U2.9 (P5.5), J2.7 (Pin_7)
- net at R12.2: now also D5.2 (A)
- net at C2.1: now also U1.10 (V3)
- net at F1.1: now also J3.A4 (VBUS), J3.A9 (VBUS), J3.B4 (VBUS), J3.B9 (VBUS)
- net at D1.1 (K): now also U1.8 (TXD)
- net at R6.2: now also U1.4 (~{RTS})
- net P1.2: now reaches U2.1 (P1.2/ADC2/SS/ECI/T2)
- net P1.2: now also J1.3 (Pin_3)
- net P3.2: now reaches U2.13 (I2CSCL_4/SCLK_4/INT0/ADC10/P3.2)
- net P3.2: now also J2.1 (Pin_1)
- net P3.3: now reaches U2.14 (I2CSDA_4/MISO_4/INT1/ADC11/P3.3)
- net P3.3: now also J2.2 (Pin_2)
- net P3.4: now reaches U2.15 (MOSI_4/CMPO/ECI_2/T1CLKO/T0/ADC12/P3.4)
- net P3.4: now also J2.3 (Pin_3)
- net P3.5: now reaches U2.16 (SS_4/CCP0_2/T0CLKO/T1/ADC13/P3.5)
- net P3.5: now also J2.4 (Pin_4)
- net P3.6: now reaches U2.17 (CMP-/CCP1_2/RxD_2/INT2/ADC14/P3.6)
- net P3.6: now also J2.5 (Pin_5)
- net P3.7: now reaches U2.18 (CMP+/CCP2/CCP2_2/TxD_2/INT3/P3.7)
- net P3.7: now also J2.6 (Pin_6)
- net P1.0: now reaches U2.19 (P1.0/ADC0/RxD2/CCP1)
- net P1.0: now also J1.1 (Pin_1)
- net P1.3: now reaches U2.2 (P1.3/ADC3/MOSI/T2CLKO)
- net P1.3: now also J1.4 (Pin_4)
- net P1.1: now reaches U2.20 (P1.1/ADC1/TxD2/CCP0)
- net P1.1: now also J1.2 (Pin_2)
- net P1.4: now reaches U2.3 (P1.4/ADC4/MISO/I2CSDA)
- net P1.4: now also J1.5 (Pin_5)
- net P1.5: now reaches U2.4 (P1.5/ADC5/SCLK/I2CSCL)
- net P1.5: now also J1.6 (Pin_6)
- net P1.6: now reaches U2.5 (P1.6/ADC6/RxD_3/MCLKO_2/XTALO)
- net P1.6: now also J1.7 (Pin_7)
- net P1.7: now reaches U2.6 (P1.7/ADC7/TxD_3/XTALI)
- net P1.7: now also J1.8 (Pin_8)
- no-connect marks 8 -> 3
Other:
- note removed: "Pins to assign:"
- moved on the sheet: C1, C2, C3, C4, D1, D2, D3, F1, Q1, Q2, R1, R10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

Commit message: Remove USER LED from schematic
Parts:
- removed D5: USER, LED_SMD:LED_0603_1608Metric, symbol Device:LED_Filled
- removed R12: 1k, Resistor_SMD:R_0603_1608Metric, symbol Device:R
Changed lines of the file:
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@@
   (junction (at 194.31 33.02) (diameter 0) (color 0 0 0 0)
-  )
-  (junction (at 140.97 135.89) (diameter 0) (color 0 0 0 0)
   )
   (junction (at 179.07 33.02) (diameter 0) (color 0 0 0 0)
@@
     (stroke (width 0) (type default))
   )
-  (wire (pts (xy 140.97 158.75) (xy 140.97 161.29))
-    (stroke (width 0) (type default))
-  )
   (wire (pts (xy 80.01 168.91) (xy 83.82 168.91))
     (stroke (width 0) (type default))
@@
     (stroke (width 0) (type default))
   )
-  (wire (pts (xy 137.16 135.89) (xy 140.97 135.89))
+  (wire (pts (xy 137.16 135.89) (xy 143.51 135.89))
     (stroke (width 0) (type default))
   )
@@
     (stroke (width 0) (type default))
   )
-  (wire (pts (xy 140.97 135.89) (xy 143.51 135.89))
-    (stroke (width 0) (type default))
-  )
   (wire (pts (xy 102.87 163.83) (xy 106.68 163.83))
     (stroke (width 0) (type default))
@@
     (stroke (width 0) (type default))
   )
-  (wire (pts (xy 140.97 151.13) (xy 140.97 149.86))
-    (stroke (width 0) (type default))
-  )
   (wire (pts (xy 134.62 30.48) (xy 134.62 31.75))
     (stroke (width 0) (type default))
@@
   )
   (wire (pts (xy 220.98 120.65) (xy 233.68 120.65))
-    (stroke (width 0) (type default))
-  )
-  (wire (pts (xy 140.97 135.89) (xy 140.97 142.24))
     (stroke (width 0) (type default))
   )
@@
     )
   )
-  (symbol (lib_id "Device:LED_Filled") (at 140.97 154.94 90) (unit 1)
-    (in_bom yes) (on_board yes) (dnp no)
-    (property "Reference" "D5" (at 144.78 153.67 90)
-      (effects (font (size 1.27 1.27)) (justify right))
-    )
-    (property "Value" "USER" (at 144.78 156.21 90)
-      (effects (font (size 1.27 1.27)) (justify right))
-    )
-    (property "Footprint" "LED_SMD:LED_0603_1608Metric" (at 140.97 154.94 0)
-      (effects (font (size 1.27 1.27)) hide)
-    )
-    (property "Datasheet" "~" (at 140.97 154.94 0)
-      (effects (font (size 1.27 1.27)) hide)
-    )
-    (pin "1")
-    (pin "2")
-    (instances
-      (project "sem-tanfolyam-stc-panel"
-        (path "/927804f4-67c2-43f0-867b-7bb7752f2aa8"
-          (reference "D5") (unit 1)
-        )
-      )
-    )
-  )
   (symbol (lib_id "power:GND") (at 104.14 78.74 0) (unit 1)
     (in_bom yes) (on_board yes) (dnp no) (fields_autoplaced)
@@
     )
   )
-  (symbol (lib_id "power:GND") (at 140.97 161.29 0) (unit 1)
-    (in_bom yes) (on_board yes) (dnp no) (fields_autoplaced)
-    (property "Reference" "#PWR023" (at 140.97 167.64 0)
-      (effects (font (size 1.27 1.27)) hide)
-    )
-    (property "Value" "GND" (at 140.97 166.37 0)
-      (effects (font (size 1.27 1.27)))
-    )
-    (property "Footprint" "" (at 140.97 161.29 0)
-      (effects (font (size 1.27 1.27)) hide)
-    )
-    (property "Datasheet" "" (at 140.97 161.29 0)
-      (effects (font (size 1.27 1.27)) hide)
-    )
-    (pin "1")
-    (instances
-      (project "sem-tanfolyam-stc-panel"
-        (path "/927804f4-67c2-43f0-867b-7bb7752f2aa8"
-          (reference "#PWR023") (unit 1)
-        )
-      )
-    )
-  )
   (symbol (lib_id "Device:D_Filled") (at 165.1 38.1 270) (unit 1)
     (in_bom yes) (on_board yes) (dnp no) (fields_autoplaced)
@@
         )
       )
-    )
-  )
-  (symbol (lib_id "Device:R") (at 140.97 146.05 0) (unit 1)
-    (in_bom yes) (on_board yes) (dnp no) (fields_autoplaced)
-    (property "Reference" "R12" (at 143.51 144.7799 0)
-      (effects (font (size 1.27 1.27)) (justify left))
-    )
-    (property "Value" "1k" (at 143.51 147.3199 0)
-      (effects (font (size 1.27 1.27)) (justify left))
-    )
-    (property "Footprint" "Resistor_SMD:R_0603_1608Metric" (at 139.192 146.05 90)
-      (effects (font (size 1.27 1.27)) hide)
-    )
-    (property "Datasheet" "~" (at 140.97 146.05 0)
-      (effects (font (size 1.27 1.27)) hide)
-    )
-    (pin "1")
-    (pin "2")
-    (instances
-      (project "sem-tanfolyam-stc-panel"
-        (path "/927804f4-67c2-43f0-867b-7bb7752f2aa8"
-          (reference "R12") (unit 1)
-        )
-      )

Commit message: BOM hozzáadva + hiányosságok meggyógyítva.
Parts:
- SW1: footprint Button_Switch_SMD:SW_Push_1P1T_NO_6x6mm_H9.5mm -> Button_Switch_SMD:SW_SPST_TL3342
Changed lines of the file:
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@@
       (effects (font (size 1.27 1.27)) (justify right))
     )
-    (property "Footprint" "Button_Switch_SMD:SW_Push_1P1T_NO_6x6mm_H9.5mm" (at 177.8 139.7 0)
+    (property "Footprint" "Button_Switch_SMD:SW_SPST_TL3342" (at 177.8 139.7 0)
       (effects (font (size 1.27 1.27)) hide)
     )

Commit message: Összemontírozva, gyártásra készen.
Parts:
- J3: footprint Connector_USB:USB_C_Receptacle_G-Switch_GT-USB-7010ASV -> jlcpcb_rotation:USB_C_Receptacle_G-Switch_GT-USB-7010ASV
- Q1, Q2: footprint Package_TO_SOT_SMD:SOT-23 -> jlcpcb_rotation:SOT-23
- U1: footprint Package_SO:MSOP-10_3x3mm_P0.5mm -> jlcpcb_rotation:MSOP-10_3x3mm_P0.5mm
- U2: footprint Package_SO:TSSOP-20_4.4x6.5mm_P0.65mm -> jlcpcb_rotation:TSSOP-20_4.4x6.5mm_P0.65mm
Changed lines of the file:
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@@
       (effects (font (size 1.27 1.27)))
     )
-    (property "Footprint" "Connector_USB:USB_C_Receptacle_G-Switch_GT-USB-7010ASV" (at 207.01 118.11 0)
+    (property "Footprint" "jlcpcb_rotation:USB_C_Receptacle_G-Switch_GT-USB-7010ASV" (at 207.01 118.11 0)
       (effects (font (size 1.27 1.27)) hide)
     )
@@
       (effects (font (size 1.27 1.27)) (justify left))
     )
-    (property "Footprint" "Package_SO:MSOP-10_3x3mm_P0.5mm" (at 90.17 64.77 0)
+    (property "Footprint" "jlcpcb_rotation:MSOP-10_3x3mm_P0.5mm" (at 90.17 64.77 0)
       (effects (font (size 1.27 1.27)) (justify left) hide)
     )
@@
       (effects (font (size 1.27 1.27)))
     )
-    (property "Footprint" "Package_TO_SOT_SMD:SOT-23" (at 206.375 30.48 0)
+    (property "Footprint" "jlcpcb_rotation:SOT-23" (at 206.375 30.48 0)
       (effects (font (size 1.27 1.27) italic) (justify left) hide)
     )
@@
       (effects (font (size 1.27 1.27)) (justify left))
     )
-    (property "Footprint" "Package_TO_SOT_SMD:SOT-23" (at 196.85 41.275 0)
+    (property "Footprint" "jlcpcb_rotation:SOT-23" (at 196.85 41.275 0)
       (effects (font (size 1.27 1.27) italic) (justify left) hide)
     )
@@
       (effects (font (size 1.27 1.27)))
     )
-    (property "Footprint" "Package_SO:TSSOP-20_4.4x6.5mm_P0.65mm" (at 62.23 130.81 0)
-      (effects (font (size 1.27 1.27)) hide)
-    )
+    (property "Footprint" "jlcpcb_rotation:TSSOP-20_4.4x6.5mm_P0.65mm" (at 62.23 130.81 0)
+      (effects (font (size 1.27 1.27)) hide)
+    )
