File: alappanel_demo/Tanfolyam_alappanel.kicad_pcb (KiCad board)
At the start: 2 copper layers, 19 parts, among them J1 Connector, J2 Connector, SW1 SW_Push, SW2 SW_Push, U1 74HC595, U3 SA39-11SRWA

Commit message: Demo projekt
Parts:
- added J3: Conn_01x09_Pin, Connector_PinHeader_2.54mm:PinHeader_1x09_P2.54mm_Vertical, F.Cu at (173.5, 107.8)
- added U4: SA39-11SRWA, Display_7Segment:Sx39-1xxxxx, F.Cu at (127.0, 80.7)
- moved C1 2.92 mm to (108.9, 106.0)
- moved J1 2.92 mm to (148.9, 87.5)
- moved J2 2.92 mm to (164.2, 107.8)
- moved R10 2.92 mm to (111.7, 89.8)
- moved R11 2.92 mm to (111.6, 84.7)
- moved R12 2.92 mm to (110.8, 80.6)
- moved R13 2.92 mm to (123.0, 95.1)
- moved R2 2.92 mm to (119.0, 114.3)
- moved R3 2.92 mm to (111.6, 112.9)
- moved R5 2.92 mm to (164.2, 83.7)
- moved R6 2.92 mm to (115.4, 95.1)
- moved R7 2.92 mm to (118.0, 95.1)
- moved R8 2.92 mm to (120.5, 95.1)
- moved R9 2.92 mm to (112.9, 95.1)
- moved SW1 2.92 mm to (128.9, 114.3)
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Routing:
- net /P1.2: track 51.0 -> 29.7 mm
- net GND: track 34.9 -> 53.6 mm
- net VCC: track 233.9 -> 239.5 mm
- net /P1.4: track 36.1 -> 34.7 mm
