File: alappanel_demo/Tanfolyam_alappanel.kicad_sch (KiCad schematic)
At the start: 19 parts, among them J1 Connector, J2 Connector, SW1 SW_Push, SW2 SW_Push, U1 74HC595, U3 SA39-11SRWA

Commit message: Demo projekt
Parts:
- added J3: Conn_01x09_Pin, Connector_PinHeader_2.54mm:PinHeader_1x09_P2.54mm_Vertical, symbol Connector:Conn_01x09_Pin
- added U4: SA39-11SRWA, Display_7Segment:Sx39-1xxxxx, symbol Display_Character:SA39-11SRWA
Connections:
- net GND: now also J3.9 (Pin_9)
- net VCC: now also J3.8 (Pin_8), U4.3 (CA), U4.8 (CA)
Other:
- note added: "0"
- note added: "1"
- note added: "2"
- note added: "3"
- note added: "QA -> D QB -> E QC -> F QD -> G QE -> DP QF -> C QG -> B QH -> A QH' X"
- note added: "QH' -> SER P1.5 -> SRCLK VCC -> ~{SRCLR} P1.2 -> RCLK GND -> ~{OE}"
- note added: "Vcc <- Termisztor [P1.4] 10k -> GND"
- note added: "Összeköttetések"
- note removed: "J3: pinheader"
- note removed: "QH' > SER P1.5 > SRCLK VCC > ~{SRCLR} P1.2 > RCLK GND > ~{OE} QA -> D QB -> E QC -> F QD -> G QE -> DP QF -> C QG -> B QH -> A QH'-> X"
- note removed: "Vcc <- Thermistor [P1.4] 10k -> GND"
