File: alappanel/Tanfolyam_alappanel.kicad_pcb (KiCad board)
At the start: 2 copper layers, 70.7 x 41.7 mm, 35 parts, among them J1 Connector, J2 Connector, J3 Connector, SW1 SW_Push, SW2 SW_Push, U1 74HC595, U2 74HC595, U3 SA39-11SRWA, U4 SA39-11SRWA

Commit message: Interaktív BOM, már a FAB rétegek feliratai is jó helyen vannak
Parts:
- D1, D2: value RED -> LED
- R1: value R -> 10k
Changed lines of the file:
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@@
 			)
 		)
-		(property "Value" "RED"
-			(at 1.27 3.96 90)
+		(property "Value" "LED"
+			(at -2.286 -0.127 0)
 			(layer "F.Fab")
 			(effects
@@
 		)
 		(property "Value" "SA39-11SRWA"
-			(at 4.44 15.716 180)
+			(at 3.81 12.954 180)
 			(layer "F.Fab")
 			(effects
@@
 		)
 		(property "Value" "Connector"
-			(at 0 23.09 180)
+			(at 2.794 10.414 -90)
 			(layer "F.Fab")
 			(effects
@@
 		)
 		(property "Value" "SA39-11SRWA"
-			(at 4.44 15.716 180)
+			(at 3.81 12.954 180)
 			(layer "F.Fab")
 			(effects
@@
 			)
 		)
-		(property "Value" "RED"
-			(at 0.73 3.96 90)
+		(property "Value" "LED"
+			(at -2.281 -0.127 180)
 			(layer "F.Fab")
 			(effects
@@
 		)
 		(property "Value" "Connector"
-			(at 0 22.65 0)
+			(at 2.794 10.517 90)
 			(layer "F.Fab")
 			(effects
@@
 		)
 		(property "Value" "1k"
-			(at 0 -1.82 -90)
+			(at 2.984 0 0)
 			(layer "B.Fab")
 			(effects
@@
 			)
 		)
-		(property "Value" "R"
+		(property "Value" "10k"
 			(at 0 -1.82 0)
 			(layer "B.Fab")
@@
 		(tags "capacitor handsolder")
 		(property "Reference" "C1"
-			(at 0 1.85 90)
+			(at 1.5625 1.905 90)
 			(layer "B.SilkS")
 			(effects
@@
 		)
 		(property "Value" "100n"
-			(at 0 -1.85 90)
+			(at -1.4855 1.905 90)
 			(layer "B.Fab")
 			(effects
@@
 		)
 		(property "Value" "1k"
-			(at 0 -1.82 0)
+			(at -3.276 0 0)
 			(layer "B.Fab")
 			(effects
@@
 		)
 		(property "Value" "1k"
-			(at 0 -1.82 0)
+			(at -3.53 0.016 0)
 			(layer "B.Fab")
 			(effects
@@
 		(tags "resistor handsolder")
 		(property "Reference" "R21"
-			(at -0.032 2.032 -90)
+			(at -1.302 2.032 -90)
 			(layer "B.SilkS")
 			(effects
@@
 		)
 		(property "Value" "1k"
-			(at 0 -1.82 -90)
+			(at 1.492 2.032 90)
 			(layer "B.Fab")
 			(effects
@@
 		(tags "resistor handsolder")
 		(property "Reference" "R11"
-			(at -0.006 -1.778 -90)
+			(at 1.01 -1.778 -90)
 			(layer "B.SilkS")
 			(effects
@@
 		)
 		(property "Value" "1k"
-			(at 0 -1.82 -90)
+			(at -1.53 -1.82 -90)
 			(layer "B.Fab")
 			(effects
@@
 		)
 		(property "Value" "1k"
-			(at 0 -1.82 -90)
+			(at 3.042 0 0)
 			(layer "B.Fab")
 			(effects
@@
 		)
 		(property "Value" "1k"
-			(at 0 -1.82 -90)
+			(at 3.042 0 0)
 			(layer "B.Fab")
 			(effects
@@
 		)
 		(property "Value" "1k"
-			(at 0 -1.82 -90)
+			(at 3.016 0 0)
 			(layer "B.Fab")
 			(effects
@@
 		(tags "resistor handsolder")
 		(property "Reference" "R16"
-			(at 0 1.82 -90)
+			(at 1.042 2.032 -90)
 			(layer "B.SilkS")
 			(effects
@@
 		)
 		(property "Value" "1k"
-			(at 0 -1.82 -90)
+			(at -1.752 2.032 -90)
 			(layer "B.Fab")
 			(effects
@@
 		)
 		(property "Value" "10k"
-			(at 0 -1.82 0)
+			(at 0 1.905 0)
 			(layer "B.Fab")
 			(effects
@@
 		)
 		(property "Value" "1k"
-			(at 0 -1.82 -90)
+			(at 2.984 0 0)
 			(layer "B.Fab")
 			(effects
@@
 		(tags "resistor handsolder")
 		(property "Reference" "R10"
-			(at 0 -1.8288 -90)
+			(at 1.0608 -1.8288 -90)
 			(layer "B.SilkS")
 			(effects
@@
 		)
 		(property "Value" "1k"
-			(at 0 -1.82 -90)
+			(at -1.4792 -1.8288 -90)
 			(layer "B.Fab")
 			(effects
@@
 		(tags "resistor handsolder")
 		(property "Reference" "R15"
-			(at 0 1.82 -90)
+			(at 1.296 1.82 -90)
 			(layer "B.SilkS")
 			(effects
@@
 		)
 		(property "Value" "1k"
-			(at 0 -1.82 -90)
+			(at -1.498 1.778 -90)
 			(layer "B.Fab")
 			(effects
@@
 		)
 		(property "Value" "1k"
-			(at 0 -1.82 -90)
+			(at 2.984 0 0)
 			(layer "B.Fab")
 			(effects
@@
 		)
 		(property "Value" "1k"
-			(at 0 -1.82 -90)
+			(at 3.042 0 0)
 			(layer "B.Fab")
 			(effects
@@
 		)
 		(property "Value" "10k"
-			(at 0 -1.82 90)
+			(at -0.736 1.778 90)
 			(layer "B.Fab")
 			(effects
@@
 		)
 		(property "Value" "1k"
-			(at 0 -1.82 -90)
+			(at 3.042 0 0)
 			(layer "B.Fab")
 			(effects
