File: stc_avr_isp/hardware/hardware.kicad_sch (KiCad schematic)
At the start: 22 parts, among them J1 Conn_01x09_Socket, J2 Conn_01x09_Socket, J3 ISP, J4 TARGET VOLTAGE, J5 BAUD RATE, U1 74HC244, U2 AMS1117-3.3

Commit message: Add fancy blink animation on reset, specify resistor values
Parts:
- C2: value 100n -> 10u
- D1: value LED_Filled -> POWER
- R5, R7: value 330 -> 1k5
- R6: value 330 -> 1k
- R9: value 330 -> 270
Other:
- note removed: "TODO: FOOTPRINTET CSEKKOLNI!"
Changed lines of the file:
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@@
 		)
 	)
-	(text "TODO: FOOTPRINTET CSEKKOLNI!"
-		(exclude_from_sim no)
-		(at 81.28 147.574 0)
-		(effects
-			(font
-				(size 2.032 2.032)
-			)
-		)
-	)
 	(label "P5.5"
 		(at 237.49 97.79 0)
@@
 			)
 		)
-		(property "Value" "330"
+		(property "Value" "1k5"
 			(at 198.12 135.8899 0)
 			(effects
@@
 			)
 		)
-		(property "Value" "LED_Filled"
+		(property "Value" "POWER"
 			(at 228.6 66.3574 90)
 			(effects
@@
 			)
 		)
-		(property "Value" "330"
+		(property "Value" "1k5"
 			(at 227.33 57.1499 0)
 			(effects
@@
 			)
 		)
-		(property "Value" "100n"
+		(property "Value" "10u"
 			(at 144.78 78.7399 0)
 			(effects
@@
 			)
 		)
-		(property "Value" "330"
+		(property "Value" "1k"
 			(at 198.12 107.9499 0)
 			(effects
@@
 			)
 		)
-		(property "Value" "330"
+		(property "Value" "270"
 			(at 228.6 93.98 90)
 			(effects
