File: stc_avr_isp/hardware_basic/hardware_basic.kicad_sch (KiCad schematic)
At the start: 16 parts, among them J1 Conn_01x09_Socket, J2 Conn_01x09_Socket, J3 ISP, J4 BAUD RATE

Commit message: Add fancy blink animation on reset, specify resistor values
Parts:
- R5, R8: value 330 -> 1k5
- R6: value 330 -> 1k
- R9: value 330 -> 270
Changed lines of the file:
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@@
 			)
 		)
-		(property "Value" "330"
+		(property "Value" "1k"
 			(at 170.18 101.5999 0)
 			(effects
@@
 			)
 		)
-		(property "Value" "330"
+		(property "Value" "1k5"
 			(at 170.18 129.5399 0)
 			(effects
@@
 			)
 		)
-		(property "Value" "330"
+		(property "Value" "1k5"
 			(at 170.18 64.7699 0)
 			(effects
@@
 			)
 		)
-		(property "Value" "330"
+		(property "Value" "270"
 			(at 199.39 87.63 90)
 			(effects
